File: pcb/PEH_PCB/PEH_PCB.kicad_sch (KiCad schematic)
At the start: 21 parts, among them J2 Conn_01x02, U1 TIP31C, U2 TIP31C, U3 TIP32C, U4 TIP32C

Commit message: spice transformer sweep and matlab get/generate figures
Parts:
- removed R2, R4: R, symbol Device:R
- L1: value L -> 15mH
Connections:
- net GND: now also L1.2, L2.2
Other:
- moved on the sheet: C1, C3, D1, D2, D4, D5, D9, J2, L1, L2, RV1, TP2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
